Commit message: adding cup holder to the robot in URDF file

File: urdf/barista_robot_model.urdf (robot description, URDF)
Before this commit: robot barista_robot, 10 links, 9 joints
Links:
- removed link chassis
- added link Cup_holder_tray_link, mass 3; collision cylinder length=0.09 radius=0.178; visual cylinder length=0.09 radius=0.178
- added link chassis_link, mass 10; collision cylinder length=0.155 radius=0.178; visual cylinder length=0.155 radius=0.178
- added link standoff_rod1_link, mass 0.5; collision cylinder length=0.22 radius=0.01; visual cylinder length=0.22 radius=0.01
- added link standoff_rod2_link, mass 0.5; collision cylinder length=0.22 radius=0.01; visual cylinder length=0.22 radius=0.01
- added link standoff_rod3_link, mass 0.5; collision cylinder length=0.22 radius=0.01; visual cylinder length=0.22 radius=0.01
- added link standoff_rod4_link, mass 0.5; collision cylinder length=0.22 radius=0.01; visual cylinder length=0.22 radius=0.01
Joints:
- added joint Cup_holder_tray_link_joint: type fixed, parent chassis_link, child Cup_holder_tray_link, origin xyz=0 0 0.3425 rpy=0 0 0
- added joint standoff_rod1_link_joint: type fixed, parent chassis_link, child standoff_rod1_link, origin xyz=0.11 0.11 0.1875 rpy=0 0 0
- added joint standoff_rod2_link_joint: type fixed, parent chassis_link, child standoff_rod2_link, origin xyz=-0.11 0.11 0.1875 rpy=0 0 0
- added joint standoff_rod3_link_joint: type fixed, parent chassis_link, child standoff_rod3_link, origin xyz=0.11 -0.11 0.1875 rpy=0 0 0
- added joint standoff_rod4_link_joint: type fixed, parent chassis_link, child standoff_rod4_link, origin xyz=-0.11 -0.11 0.1875 rpy=0 0 0
- joint back_yaw_joint: parent chassis -> chassis_link
- joint base_link_joint: child chassis -> chassis_link
- joint front_yaw_joint: parent chassis -> chassis_link
- joint joint_left_wheel: parent chassis -> chassis_link
- joint joint_right_wheel: parent chassis -> chassis_link

Commit message: adding laser scan to urdf file

File: urdf/barista_robot_model.urdf (robot description, URDF)
Before this commit: robot barista_robot, 15 links, 14 joints
Links:
- added link laser_scan_model_link, mass 0.01; collision cylinder length=0.0408 radius=0.037493; visual mesh filename=package://barista_robot_description/meshes/sensors/hokuyo_u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 scale=1.0 1.0 1.0
Joints:
- added joint laser_scan_model_link_joint: type continuous, parent chassis_link, child laser_scan_model_link, origin xyz=0.1 0.0 0.0775 rpy=0 0 0, axis 0 0 1, limit effort=10.0 velocity=2.0

Commit message: fix laser scan

File: urdf/barista_robot_model.urdf (robot description, URDF)
Before this commit: robot barista_robot, 16 links, 15 joints
Links:
- removed link laser_scan_model_link
- added link laser_model_link, mass 0.01; collision mesh filename=package://barista_robot_description/meshes/sensors/hokuyo_u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 scale=1.0 1.0 1.0; visual mesh filename=package://barista_robot_description/meshes/sensors/hokuyo_u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 scale=1.0 1.0 1.0
- added link laser_scan_frame
Joints:
- added joint laser_scan_frame_joint: type fixed, parent laser_model_link, child laser_scan_frame, origin xyz=0 0 0.05 rpy=0 0 0
- joint laser_scan_model_link_joint: axis 0 0 1 -> 0 0 0; child laser_scan_model_link -> laser_model_link; limit effort=10.0 velocity=2.0 -> (none); type continuous -> fixed

Commit message: part 1 completed

File: urdf/barista_robot_model.urdf (robot description, URDF)
Before this commit: robot barista_robot, 17 links, 16 joints
Links:
- link Cup_holder_tray_link: mass 3 -> 2
- link chassis_link: mass 10 -> 5
- link standoff_rod1_link: mass 0.5 -> 0.1
- link standoff_rod2_link: mass 0.5 -> 0.1
- link standoff_rod3_link: mass 0.5 -> 0.1
- link standoff_rod4_link: mass 0.5 -> 0.1
