Commit message: adding inertial calculation in xacros files

File: xacro/barista_robot_model.urdf.xacro (robot description, xacro)
@@ -7,4 +7,6 @@
 <xacro:property name="body_radius" value="0.178"/>
 <xacro:property name="body_height" value="0.155"/>
+<xacro:property name="body_mass"   value= "5"/>
+<xacro:property name="wheel_separation" value = "0.3"/>
   <material name="red">
     <color rgba="1.0 0.0 0.0 1"/>
@@ -41,6 +43,9 @@
     </collision>
     <inertial>
-      <mass value="5"/>
-      <inertia ixx="0.04961541667" ixy="0" ixz="0" iyy="0.04961541667" iyz="0" izz="0.04961541667"/>
+      <mass value="${body_mass}"/>
+      <!-- <inertia ixx="0.04961541667" ixy="0" ixz="0" iyy="0.04961541667" iyz="0" izz="0.04961541667"/> -->
+      <inertia  ixx="${body_mass*(3*body_radius*body_radius+body_height*body_height)/12}" ixy = "0" ixz = "0"
+            iyy="${body_mass*(3*body_radius*body_radius+body_height*body_height)/12}" iyz = "0"
+            izz="${body_mass*(body_radius*body_radius)/2}" />
     </inertial>
   </link>
@@ -49,5 +54,5 @@
   </gazebo>
   <joint name="base_link_joint" type="fixed">
-    <origin rpy="0 0 0" xyz="0 0 0.0775" />
+    <origin rpy="0 0 0" xyz="0 0 ${body_height/2}" />
     <parent link="base_link" />
     <child link="chassis_link" />
@@ -65,5 +70,5 @@
   </gazebo>
   <joint name="standoff_rod1_link_joint" type="fixed">
-    <origin rpy="0 0 0" xyz="0.11 0.11 0.1875" />
+    <origin rpy="0 0 0" xyz="${body_radius*0.618} ${body_radius*0.618} ${standoff_height/2+body_height/2}" />
     <parent link="chassis_link" />
     <child link="standoff_rod1_link" />
@@ -73,5 +78,5 @@
   </gazebo>
   <joint name="standoff_rod2_link_joint" type="fixed">
-    <origin rpy="0 0 0" xyz="-0.11 0.11 0.1875" />
+    <origin rpy="0 0 0" xyz="-${body_radius*0.618} ${body_radius*0.618} ${standoff_height/2+body_height/2}" />
     <parent link="chassis_link" />
     <child link="standoff_rod2_link" />
@@ -81,5 +86,5 @@
   </gazebo>
   <joint name="standoff_rod3_link_joint" type="fixed">
-    <origin rpy="0 0 0" xyz="0.11 -0.11 0.1875" />
+    <origin rpy="0 0 0" xyz="${body_radius*0.618} -${body_radius*0.618} ${standoff_height/2+body_height/2}" />
     <parent link="chassis_link" />
     <child link="standoff_rod3_link" />
@@ -89,5 +94,5 @@
   </gazebo>
   <joint name="standoff_rod4_link_joint" type="fixed">
-    <origin rpy="0 0 0" xyz="-0.11 -0.11 0.1875" />
+    <origin rpy="0 0 0" xyz="-${body_radius*0.618} -${body_radius*0.618} ${standoff_height/2+body_height/2}" />
     <parent link="chassis_link" />
     <child link="standoff_rod4_link" />
@@ -99,5 +104,5 @@
   </gazebo>
   <joint name="Cup_holder_tray_link_joint" type="fixed">
-    <origin rpy="0 0 0" xyz="0 0 0.3425" />
+    <origin rpy="0 0 0" xyz="0 0 ${body_height/2+standoff_height+cup_holde_tray_height/2}" />
     <parent link="chassis_link" />
     <child link="Cup_holder_tray_link" />
@@ -115,5 +120,5 @@
   </gazebo>
   <joint name="joint_left_wheel" type="continuous">
-    <origin rpy="0 0 0" xyz="0 0.15 -0.06"/>
+    <origin rpy="0 0 0" xyz="0 ${wheel_separation/2} -0.06"/>
     <child link="left_wheel"/>
     <parent link="chassis_link"/>
@@ -130,5 +135,5 @@
   </gazebo>
   <joint name="joint_right_wheel" type="continuous">
-    <origin rpy="0 0 0" xyz="0 -0.15 -0.06"/>
+    <origin rpy="0 0 0" xyz="0 -${wheel_separation/2} -0.06"/>
     <child link="right_wheel"/>
     <parent link="chassis_link"/>
@@ -357,6 +362,6 @@
       <right_joint>joint_right_wheel</right_joint>
       <!-- kinematics -->
-      <wheel_separation>0.3</wheel_separation>
-      <wheel_diameter>0.0704</wheel_diameter>
+      <wheel_separation>${wheel_separation}</wheel_separation>
+      <wheel_diameter>${wheel_radius*2}</wheel_diameter>
       <!-- limits -->
       <max_wheel_torque>1.0</max_wheel_torque>

File: xacro/cup_holder_tray.xacro (robot description, xacro)
@@ -3,4 +3,5 @@
 <xacro:property name="cup_holde_tray_radius" value="0.178"/>
 <xacro:property name="cup_holde_tray_height" value="0.09"/>
+<xacro:property name="cup_holde_tray_mass" value="2"/>
 <!-- Cup holder tray -->
 <xacro:macro name="Cup_holder_tray" params="Cup_holder_tray_name">
@@ -18,6 +19,9 @@
     </collision>
     <inertial>
-      <mass value="2"/>
-      <inertia ixx="0.005064" ixy="0" ixz="0" iyy="0.005064" iyz="0" izz="0.0081"/>
+      <mass value="${cup_holde_tray_mass}"/>
+      <!-- <inertia ixx="0.005064" ixy="0" ixz="0" iyy="0.005064" iyz="0" izz="0.0081"/> -->
+      <inertia  ixx="${cup_holde_tray_mass*(3*cup_holde_tray_radius*cup_holde_tray_radius+cup_holde_tray_height*cup_holde_tray_height)/12}" ixy = "0" ixz = "0"
+            iyy="${cup_holde_tray_mass*(3*cup_holde_tray_radius*cup_holde_tray_radius+cup_holde_tray_height*cup_holde_tray_height)/12}" iyz = "0"
+            izz="${cup_holde_tray_mass*(cup_holde_tray_radius*cup_holde_tray_radius)/2}" />
     </inertial>
   </link>

File: xacro/standoff.xacro (robot description, xacro)
@@ -3,4 +3,5 @@
 <xacro:property name="standoff_radius" value="0.01"/>
 <xacro:property name="standoff_height" value="0.22"/>
+<xacro:property name="standoff_mass" value="0.1"/>
 <!-- standoff rods macro -->
 <xacro:macro name="standoff" params="standoff_rod_name">
@@ -18,6 +19,9 @@
     </collision>
     <inertial>
-      <mass value="0.1"/>
-      <inertia ixx="0.0006533333333" ixy="0" ixz="0" iyy="0.0006533333333" iyz="0" izz="0.0005"/>
+      <mass value="${standoff_mass}"/>
+      <!-- <inertia ixx="0.0006533333333" ixy="0" ixz="0" iyy="0.0006533333333" iyz="0" izz="0.0005"/> -->
+      <inertia  ixx="${standoff_mass*(3*standoff_radius*standoff_radius+standoff_height*standoff_height)/12}" ixy = "0" ixz = "0"
+            iyy="${standoff_mass*(3*standoff_radius*standoff_radius+standoff_height*standoff_height)/12}" iyz = "0"
+            izz="${standoff_mass*(standoff_radius*standoff_radius)/2}" />
     </inertial>
   </link>

File: xacro/wheel.xacro (robot description, xacro)
@@ -3,4 +3,5 @@
 <xacro:property name="wheel_width" value="0.0206"/>
 <xacro:property name="wheel_radius" value="0.0352"/>
+<xacro:property name="wheel_mass" value="2"/>
 <!-- Wheel Left -->
 <xacro:macro name="wheel" params="wheel_name">
@@ -21,6 +22,9 @@
       <inertial>
         <origin rpy="0 1.5707 1.5707" xyz="0 0 0"/>
-        <mass value="2"/>
-        <inertia ixx="0.000690247" ixy="0" ixz="0" iyy="0.000690247" iyz="0" izz="0.00123904"/>
+        <mass value="${wheel_mass}"/>
+        <!-- <inertia ixx="0.000690247" ixy="0" ixz="0" iyy="0.000690247" iyz="0" izz="0.00123904"/> -->
+        <inertia  ixx="${wheel_mass*(3*wheel_radius*wheel_radius+wheel_width*wheel_width)/12}" ixy = "0" ixz = "0"
+        iyy="${wheel_mass*(3*wheel_radius*wheel_radius+wheel_width*wheel_width)/12}" iyz = "0"
+        izz="${wheel_mass*(wheel_radius*wheel_radius)/2}" />
       </inertial>
   </link>

Commit message: updating some valuse for inertial to make the robot more stable

File: xacro/barista_robot_model.urdf.xacro (robot description, xacro)
@@ -159,6 +159,6 @@
       <inertial>
           <origin rpy="0 1.5707 1.5707" xyz="0 0 0"/>
-          <mass value="0.001"/>
-          <inertia ixx="5.145833333333334e-09" ixy="0" ixz="0" iyy="5.145833333333334e-09" iyz="0" izz="1.0125000000000003e-08"/>
+          <mass value="0.01"/>
+          <inertia ixx="0.0000008665583333" ixy="0" ixz="0" iyy="0.0000008665583333" iyz="0" izz="0.00000156645"/>
       </inertial>
   </link>
@@ -190,6 +190,6 @@
       <inertial>
           <origin rpy="0 1.5707 1.5707" xyz="0 0 0"/>
-          <mass value="0.001"/>
-          <inertia ixx="5.145833333333334e-09" ixy="0" ixz="0" iyy="5.145833333333334e-09" iyz="0" izz="1.0125000000000003e-08"/>
+          <mass value="0.01"/>
+          <inertia ixx="0.0000008665583333" ixy="0" ixz="0" iyy="0.0000008665583333" iyz="0" izz="0.00000156645"/>
       </inertial>
   </link>
@@ -221,6 +221,6 @@
     <inertial>
         <origin rpy="0 1.5707 1.5707" xyz="0 0 0"/>
-        <mass value="0.001"/>
-        <inertia ixx="4e-08" ixy="0" ixz="0" iyy="4e-08" iyz="0" izz="4e-08"/>
+        <mass value="0.1"/>
+        <inertia ixx="0.00000125316" ixy="0" ixz="0" iyy="0.00000125316" iyz="0" izz="0.00000125316"/>
     </inertial>
   </link>
@@ -257,6 +257,6 @@
       <inertial>
           <origin rpy="0 1.5707 1.5707" xyz="0 0 0"/>
-          <mass value="0.001"/>
-          <inertia ixx="5.145833333333334e-09" ixy="0" ixz="0" iyy="5.145833333333334e-09" iyz="0" izz="1.0125000000000003e-08"/>
+          <mass value="0.01"/>
+          <inertia ixx="0.0000008665583333" ixy="0" ixz="0" iyy="0.000008665583333" iyz="0" izz="0.00000156645"/>
       </inertial>
   </link>
@@ -288,6 +288,6 @@
       <inertial>
           <origin rpy="0 1.5707 1.5707" xyz="0 0 0"/>
-          <mass value="0.001"/>
-          <inertia ixx="5.145833333333334e-09" ixy="0" ixz="0" iyy="5.145833333333334e-09" iyz="0" izz="1.0125000000000003e-08"/>
+          <mass value="0.01"/>
+          <inertia ixx="0.0000008665583333" ixy="0" ixz="0" iyy="0.0000008665583333" iyz="0" izz="0.00000156645"/>
       </inertial>
   </link>
@@ -319,6 +319,6 @@
     <inertial>
         <origin rpy="0 1.5707 1.5707" xyz="0 0 0"/>
-        <mass value="0.001"/>
-        <inertia ixx="4e-08" ixy="0" ixz="0" iyy="4e-08" iyz="0" izz="4e-08"/>
+        <mass value="0.01"/>
+        <inertia ixx="0.00000125316" ixy="0" ixz="0" iyy="0.0000125316" iyz="0" izz="0.00000125316"/>
     </inertial>
   </link>

File: xacro/standoff.xacro (robot description, xacro)
@@ -3,5 +3,5 @@
 <xacro:property name="standoff_radius" value="0.01"/>
 <xacro:property name="standoff_height" value="0.22"/>
-<xacro:property name="standoff_mass" value="0.1"/>
+<xacro:property name="standoff_mass" value="0.2"/>
 <!-- standoff rods macro -->
 <xacro:macro name="standoff" params="standoff_rod_name">

Commit message: spawn two robots

File: xacro/barista_robot_model.urdf.xacro (robot description, xacro)
@@ -1,4 +1,5 @@
 <?xml version="1.0"?>
 <robot xmlns:xacro="http://www.ros.org/wiki/xacro"  name="barista_robot">
+<xacro:property name="robot_name" value="$(arg robot_name)"/>
 <xacro:include filename="$(find barista_robot_description)/xacro/wheel.xacro" />
 <xacro:include filename="$(find barista_robot_description)/xacro/standoff.xacro" />
@@ -342,4 +343,5 @@
     <plugin name="barisat_robot_joint_state" filename="libgazebo_ros_joint_state_publisher.so">
       <ros>
+          <namespace>/${robot_name}</namespace>
           <remapping>~/out:=joint_states</remapping>
       </ros>
@@ -358,4 +360,8 @@
   <gazebo>
     <plugin filename="libgazebo_ros_diff_drive.so" name="differential_drive_controller">
+      <ros>
+        <namespace>/${robot_name}</namespace>
+        <remapping>/out:=cmd_vel</remapping>
+      </ros>
       <!-- wheels -->
       <left_joint>joint_left_wheel</left_joint>
@@ -370,6 +376,6 @@
       <publish_odom>true</publish_odom>
       <publish_odom_tf>true</publish_odom_tf>
-      <odometry_frame>odom</odometry_frame>
-      <robot_base_frame>base_link</robot_base_frame>
+      <odometry_frame>${robot_name}/odom</odometry_frame>
+      <robot_base_frame>${robot_name}/base_link</robot_base_frame>
     </plugin>
   </gazebo>
@@ -429,9 +435,10 @@
         <visualize>true</visualize>
         <update_rate>100.0</update_rate>
-        <plugin name="laser_scan_node" filename="libgazebo_ros_ray_sensor.so">
+        <plugin name="${robot_name}_laser_scan_node" filename="libgazebo_ros_ray_sensor.so">
           <ros>
+            <namespace>/${robot_name}</namespace>
             <remapping>~/out:=scan</remapping>
           </ros>
-          <frame_name>laser_scan_frame</frame_name>
+          <frame_name>${robot_name}/laser_scan_frame</frame_name>
           <output_type>sensor_msgs/LaserScan</output_type>
         </plugin>

Commit message: change the color of each robot

File: xacro/barista_robot_model.urdf.xacro (robot description, xacro)
@@ -2,4 +2,12 @@
 <robot xmlns:xacro="http://www.ros.org/wiki/xacro"  name="barista_robot">
 <xacro:property name="robot_name" value="$(arg robot_name)"/>
+<xacro:if value="${robot_name == 'rick'}">
+    <xacro:property name="robot_color_rviz" value="blue"/>
+    <xacro:property name="robot_color_gazebo" value="Gazebo/Blue"/>
+</xacro:if>
+<xacro:unless value="${robot_name == 'rick'}">
+    <xacro:property name="robot_color_rviz" value="red"/>
+    <xacro:property name="robot_color_gazebo" value="Gazebo/Red"/>
+</xacro:unless>
 <xacro:include filename="$(find barista_robot_description)/xacro/wheel.xacro" />
 <xacro:include filename="$(find barista_robot_description)/xacro/standoff.xacro" />
@@ -36,5 +44,5 @@
             <cylinder radius="${body_radius}" length="${body_height}"/>
         </geometry>
-		<material name="blue"/>
+		<material name="${robot_color_rviz}"/>
     </visual>
     <collision>
@@ -52,5 +60,5 @@
   </link>
 	<gazebo reference="chassis_link">
-      <material>Gazebo/Blue</material>
+      <material>${robot_color_gazebo}</material>
   </gazebo>
   <joint name="base_link_joint" type="fixed">
@@ -102,5 +110,5 @@
 <xacro:Cup_holder_tray    Cup_holder_tray_name="Cup_holder_tray_link"/>
   <gazebo reference="Cup_holder_tray_link">
-      <material>Gazebo/Blue</material>
+      <material>${robot_color_gazebo}</material>
   </gazebo>
   <joint name="Cup_holder_tray_link_joint" type="fixed">
@@ -435,5 +443,5 @@
         <visualize>true</visualize>
         <update_rate>100.0</update_rate>
-        <plugin name="${robot_name}_laser_scan_node" filename="libgazebo_ros_ray_sensor.so">
+        <plugin name="laser_scan_node" filename="libgazebo_ros_ray_sensor.so">
           <ros>
             <namespace>/${robot_name}</namespace>

File: xacro/cup_holder_tray.xacro (robot description, xacro)
@@ -11,5 +11,5 @@
             <cylinder radius="${cup_holde_tray_radius}" length="${cup_holde_tray_height}"/>
         </geometry>
-		<material name="blue"/>
+		<material name="${robot_color_rviz}"/>
     </visual>
     <collision>

Commit message: fix robot model in rviz

File: xacro/barista_robot_model.urdf.xacro (robot description, xacro)
@@ -1,21 +1,21 @@
 <?xml version="1.0"?>
 <robot xmlns:xacro="http://www.ros.org/wiki/xacro"  name="barista_robot">
-<xacro:property name="robot_name" value="$(arg robot_name)"/>
-<xacro:if value="${robot_name == 'rick'}">
-    <xacro:property name="robot_color_rviz" value="blue"/>
-    <xacro:property name="robot_color_gazebo" value="Gazebo/Blue"/>
-</xacro:if>
-<xacro:unless value="${robot_name == 'rick'}">
-    <xacro:property name="robot_color_rviz" value="red"/>
-    <xacro:property name="robot_color_gazebo" value="Gazebo/Red"/>
-</xacro:unless>
-<xacro:include filename="$(find barista_robot_description)/xacro/wheel.xacro" />
-<xacro:include filename="$(find barista_robot_description)/xacro/standoff.xacro" />
-<xacro:include filename="$(find barista_robot_description)/xacro/cup_holder_tray.xacro" />
-<xacro:arg  name="include_laser" default="true"/>
-<xacro:property name="body_radius" value="0.178"/>
-<xacro:property name="body_height" value="0.155"/>
-<xacro:property name="body_mass"   value= "5"/>
-<xacro:property name="wheel_separation" value = "0.3"/>
+    <xacro:property name="robot_name" value="$(arg robot_name)"/>
+    <xacro:if value="${robot_name == 'rick'}">
+        <xacro:property name="robot_color_rviz" value="blue"/>
+        <xacro:property name="robot_color_gazebo" value="Gazebo/Blue"/>
+    </xacro:if>
+    <xacro:unless value="${robot_name == 'rick'}">
+        <xacro:property name="robot_color_rviz" value="red"/>
+        <xacro:property name="robot_color_gazebo" value="Gazebo/Red"/>
+    </xacro:unless>
+    <xacro:include filename="$(find barista_robot_description)/xacro/wheel.xacro" />
+    <xacro:include filename="$(find barista_robot_description)/xacro/standoff.xacro" />
+    <xacro:include filename="$(find barista_robot_description)/xacro/cup_holder_tray.xacro" />
+    <xacro:arg  name="include_laser" default="true"/>
+    <xacro:property name="body_radius" value="0.178"/>
+    <xacro:property name="body_height" value="0.155"/>
+    <xacro:property name="body_mass"   value= "5"/>
+    <xacro:property name="wheel_separation" value = "0.3"/>
   <material name="red">
     <color rgba="1.0 0.0 0.0 1"/>
@@ -59,7 +59,7 @@
     </inertial>
   </link>
-	<gazebo reference="chassis_link">
+   <gazebo reference="chassis_link">
       <material>${robot_color_gazebo}</material>
-  </gazebo>
+   </gazebo>
   <joint name="base_link_joint" type="fixed">
     <origin rpy="0 0 0" xyz="0 0 ${body_height/2}" />

Commit message: update inertial

File: xacro/barista_robot_model.urdf.xacro (robot description, xacro)
@@ -168,6 +168,6 @@
       <inertial>
           <origin rpy="0 1.5707 1.5707" xyz="0 0 0"/>
-          <mass value="0.01"/>
-          <inertia ixx="0.0000008665583333" ixy="0" ixz="0" iyy="0.0000008665583333" iyz="0" izz="0.00000156645"/>
+          <mass value="0.1"/>
+          <inertia ixx="0.000008665583333" ixy="0" ixz="0" iyy="0.000008665583333" iyz="0" izz="0.0000156645"/>
       </inertial>
   </link>
@@ -231,5 +231,5 @@
         <origin rpy="0 1.5707 1.5707" xyz="0 0 0"/>
         <mass value="0.1"/>
-        <inertia ixx="0.00000125316" ixy="0" ixz="0" iyy="0.00000125316" iyz="0" izz="0.00000125316"/>
+        <inertia ixx="0.0000125316" ixy="0" ixz="0" iyy="0.0000125316" iyz="0" izz="0.0000125316"/>
     </inertial>
   </link>
@@ -266,6 +266,6 @@
       <inertial>
           <origin rpy="0 1.5707 1.5707" xyz="0 0 0"/>
-          <mass value="0.01"/>
-          <inertia ixx="0.0000008665583333" ixy="0" ixz="0" iyy="0.000008665583333" iyz="0" izz="0.00000156645"/>
+          <mass value="0.1"/>
+          <inertia ixx="0.000008665583333" ixy="0" ixz="0" iyy="0.000008665583333" iyz="0" izz="0.0000156645"/>
       </inertial>
   </link>
@@ -297,6 +297,6 @@
       <inertial>
           <origin rpy="0 1.5707 1.5707" xyz="0 0 0"/>
-          <mass value="0.01"/>
-          <inertia ixx="0.0000008665583333" ixy="0" ixz="0" iyy="0.0000008665583333" iyz="0" izz="0.00000156645"/>
+          <mass value="0.1"/>
+          <inertia ixx="0.000008665583333" ixy="0" ixz="0" iyy="0.000008665583333" iyz="0" izz="0.0000156645"/>
       </inertial>
   </link>
@@ -328,6 +328,6 @@
     <inertial>
         <origin rpy="0 1.5707 1.5707" xyz="0 0 0"/>
-        <mass value="0.01"/>
-        <inertia ixx="0.00000125316" ixy="0" ixz="0" iyy="0.0000125316" iyz="0" izz="0.00000125316"/>
+        <mass value="0.1"/>
+        <inertia ixx="0.0000125316" ixy="0" ixz="0" iyy="0.0000125316" iyz="0" izz="0.0000125316"/>
     </inertial>
   </link>

Commit message: update inertial

File: xacro/barista_robot_model.urdf.xacro (robot description, xacro)
@@ -168,6 +168,6 @@
       <inertial>
           <origin rpy="0 1.5707 1.5707" xyz="0 0 0"/>
-          <mass value="0.1"/>
-          <inertia ixx="0.000008665583333" ixy="0" ixz="0" iyy="0.000008665583333" iyz="0" izz="0.0000156645"/>
+          <mass value="0.01"/>
+          <inertia ixx="0.0000008665583333" ixy="0" ixz="0" iyy="0.0000008665583333" iyz="0" izz="0.00000156645"/>
       </inertial>
   </link>
@@ -230,6 +230,6 @@
     <inertial>
         <origin rpy="0 1.5707 1.5707" xyz="0 0 0"/>
-        <mass value="0.1"/>
-        <inertia ixx="0.0000125316" ixy="0" ixz="0" iyy="0.0000125316" iyz="0" izz="0.0000125316"/>
+        <mass value="0.01"/>
+        <inertia ixx="0.00000125316" ixy="0" ixz="0" iyy="0.00000125316" iyz="0" izz="0.00000125316"/>
     </inertial>
   </link>
@@ -266,6 +266,6 @@
       <inertial>
           <origin rpy="0 1.5707 1.5707" xyz="0 0 0"/>
-          <mass value="0.1"/>
-          <inertia ixx="0.000008665583333" ixy="0" ixz="0" iyy="0.000008665583333" iyz="0" izz="0.0000156645"/>
+          <mass value="0.01"/>
+          <inertia ixx="0.0000008665583333" ixy="0" ixz="0" iyy="0.0000008665583333" iyz="0" izz="0.00000156645"/>
       </inertial>
   </link>
@@ -297,6 +297,6 @@
       <inertial>
           <origin rpy="0 1.5707 1.5707" xyz="0 0 0"/>
-          <mass value="0.1"/>
-          <inertia ixx="0.000008665583333" ixy="0" ixz="0" iyy="0.000008665583333" iyz="0" izz="0.0000156645"/>
+          <mass value="0.01"/>
+          <inertia ixx="0.0000008665583333" ixy="0" ixz="0" iyy="0.0000008665583333" iyz="0" izz="0.00000156645"/>
       </inertial>
   </link>
@@ -328,6 +328,6 @@
     <inertial>
         <origin rpy="0 1.5707 1.5707" xyz="0 0 0"/>
-        <mass value="0.1"/>
-        <inertia ixx="0.0000125316" ixy="0" ixz="0" iyy="0.0000125316" iyz="0" izz="0.0000125316"/>
+        <mass value="0.01"/>
+        <inertia ixx="0.00000125316" ixy="0" ixz="0" iyy="0.00000125316" iyz="0" izz="0.00000125316"/>
     </inertial>
   </link>
